File: OwlClock2.brd (EAGLE design)
At the start: 160 x 54.6 mm, 98 parts, among them IC1 MCP1703DB, J1 AVR_SPI_PRG_6NS, J2 POWER_JACKPTH, Q1 16Mhz, U1 ATMEGA328P_PDIP

Commit message: Fix problem where real time clock was connected to the wrong supply
Connections:
- net VCC: no longer JP1.5
- net VSS: now also JP1.5
Routing:
- net VSS: track 100.4 -> 132.2 mm
Other:
- board text added: "V2.0"
- board text removed: "V1.0"
Changed lines of the file:
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@@
 <text x="134.239" y="68.199" size="1.016" layer="21">32K</text>
 <text x="110.49" y="52.07" size="1.4224" layer="21">Owl Clock</text>
-<text x="110.49" y="49.53" size="1.4224" layer="21">V1.0</text>
+<text x="110.49" y="49.53" size="1.4224" layer="21">V2.0</text>
 </plain>
 <attributes>
@@
 <signal name="VCC">
 <contactref element="J2" pad="PWR"/>
-<contactref element="JP1" pad="5"/>
 <contactref element="TENS1:C1" pad="1"/>
 <contactref element="TENS1:D1" pad="1"/>
@@
 <contactref element="C6" pad="2"/>
 <wire x1="58.42" y1="58.42" x2="58" y2="58.42" width="0.4064" layer="1"/>
+<contactref element="JP1" pad="5"/>
+<wire x1="106.68" y1="60.96" x2="102.87" y2="57.15" width="0.4064" layer="16"/>
+<wire x1="128.27" y1="60.96" x2="106.68" y2="60.96" width="0.4064" layer="16"/>
+<wire x1="130.81" y1="58.42" x2="128.27" y2="60.96" width="0.4064" layer="16"/>
+<wire x1="132.08" y1="58.42" x2="130.81" y2="58.42" width="0.4064" layer="16"/>
 </signal>
 <signal name="N$4">
