File: OwlClock2.brd (EAGLE design)
At the start: 160 x 54.6 mm, 98 parts, among them IC1 MCP1703DB, J1 AVR_SPI_PRG_6NS, J2 POWER_JACKPTH, Q1 16Mhz, U1 ATMEGA328P_PDIP

Commit message: Finally add the owlLogo to the boards and add a regulator bypass block.
Parts:
- added SUPPLY_BYPASS: M02LOCK, SparkFun-Connectors:1X02_LOCK
Connections:
- net VCC: now also SUPPLY_BYPASS.2
- net VSS: now also SUPPLY_BYPASS.1
Routing:
- net VSS: track 132.2 -> 139.5 mm
Other:
- board text added: "/Users/kschaefer/Documents/owl-clock/owlLogoMono3.BMP"
- board text added: "BYPASS"
- board text added: "EYE INSIDE"
- board text added: "EYE TOP"
- board text removed: "/Users/kschaefer/Documents/OwlLogoMono.bmp"
- board text removed: "PHOTO INSIDE"
